File: BatteryBox.kicad_sch (KiCad schematic)
At the start: 0 parts

Commit message: Add files via upload
Finished everything except for the micro schematic
Parts:
- added BT1, BT2, BT3: 1.5V, symbol Device:Battery_Cell
- added D1: D, symbol Device:D
- added J1: Conn_01x02_Socket, symbol Connector:Conn_01x02_Socket
- added J2: Conn_01x02_Pin, symbol Connector:Conn_01x02_Pin
Connections:
- new net: BT3.2 (-), J1.1 (Pin_1)
- new net: BT1.1 (+), J1.2 (Pin_2)
- new net: BT2.2 (-), BT3.1 (+)
- new net: BT1.2 (-), BT2.1 (+)
- new net: D1.2 (A), J2.2 (Pin_2)
- new net Boost Vin (V+): D1.1 (K)
- new net Boost Vout (V-): J2.1 (Pin_1)
Other:
- note added: "Battery "Box""
- note added: "Edge of PCB Board"
