File: GPS.kicad_sch (KiCad schematic)
At the start: 0 parts

Commit message: Updated the indivdual components.
Some of the individual components still need to be updated and completed. With the battery box, include the diode. The full schematic is not the update one as Andrew has the updated one with the correct flyback diode placement.
Parts:
- added U10: FGPMMOPA6H, GPS Module:FGPMMOPA6H, symbol Adafruit Ultimate GPS Hat-eagle-import:GPS_FGPMMOPA6H
Connections:
- new net Buck Boost Pin One (Vout): U10.P$1 (VCC), U10.P$4 (VBACKUP)
- new net Earth: U10.P$12 (GND@3), U10.P$19 (GND@4), U10.P$3 (GND@1), U10.P$8 (GND@2)
- new net Micro UART RX PA1 (Pin 15): U10.P$9 (TX)
- new net Micro UART TX PA0 (Pin 14): U10.P$10 (RX)
Other:
- note added: "GPS"

Commit message: Add files via upload
Finished everything except for the micro schematic
Changed lines of the file:
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@@
 		(color 0 0 0 0)
 	)
+	(junction
+		(at 160.02 88.9)
+		(diameter 0)
+		(color 0 0 0 0)
+	)
 	(wire
 		(pts
@@
 		(pts
 			(xy 72.39 104.14) (xy 72.39 135.89)
+		)
+		(stroke
+			(width 0)
+			(type default)
+		)
+	)
+	(wire
+		(pts
+			(xy 160.02 78.74) (xy 160.02 88.9)
 		)
 		(stroke
@@
 				(hide yes)
 			)
+		)
+	)
+	(global_label "Buck Boost Ground (V-)"
+		(shape input)
+		(at 160.02 78.74 0)
+		(fields_autoplaced yes)
+		(effects
+			(font
+				(size 1.27 1.27)
+				(bold yes)
+			)
+			(justify left)
+		)
+		(property "Intersheetrefs" "${INTERSHEET_REFS}"
+			(at 187.2481 78.74 0)
+			(effects
+				(font
+					(size 1.27 1.27)
+				)
+				(justify left)
+				(hide yes)
+			)
