File: Boost.kicad_sch (KiCad schematic)
At the start: 0 parts

Commit message: Updated the indivdual components.
Some of the individual components still need to be updated and completed. With the battery box, include the diode. The full schematic is not the update one as Andrew has the updated one with the correct flyback diode placement.
Parts:
- added C13: 10 uF, 3 mOhms, symbol Device:C
- added C4: 1.8 nF, symbol Device:C
- added C5: 22 uF, 1 mOhms, symbol Device:C
- added D3: 320 mV, 2A, symbol Device:D_Schottky
- added L2: 3.3 uH, 20 Ohm, symbol Device:L
- added R1, R2: 10k Ohms, symbol Device:R_US
- added R3: 30k Ohms, symbol Device:R_US
- added U11: LM2735X, Boost Converter Chip:MF05A, symbol 2024-09-27_13-12-28-eagle-import:LM2735XMF/NOPBLM2735XMF/NOPB
Connections:
- new net: C4.1, R2.1, R3.1, U11.3 (FB@4)
- new net: C4.2, C5.1, D3.1 (K), R3.2
- new net: D3.2 (A), L2.2, U11.1 (SW@3)
- new net: R1.2, U11.4 (EN@2)
- new net Battery Box Vout (Flyback Diode): C13.1, L2.1, R1.1, U11.5 (VIN@1)
- new net Earth: C13.2, C5.2, R2.2, U11.2 (GND@5)

Commit message: Add files via upload
Finished everything except for the micro schematic
Connections:
- net Boost Output (Vout): now reaches C4.2, C5.1, D3.1 (K), R3.2
Changed lines of the file:
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@@
+	)
+	(junction
+		(at 184.15 121.92)
+		(diameter 0)
+		(color 0 0 0 0)
+	)
+	(junction
+		(at 184.15 60.96)
+		(diameter 0)
+		(color 0 0 0 0)
 	)
 	(junction
@@
 	)
 	(junction
+		(at 69.85 121.92)
+		(diameter 0)
+		(color 0 0 0 0)
+	)
+	(junction
 		(at 86.36 60.96)
 		(diameter 0)
@@
 	(wire
 		(pts
+			(xy 69.85 121.92) (xy 34.29 121.92)
+		)
+		(stroke
+			(width 0)
+			(type default)
+		)
+	)
+	(wire
+		(pts
+			(xy 184.15 121.92) (xy 208.28 121.92)
+		)
+		(stroke
+			(width 0)
+			(type default)
+		)
+	)
+	(wire
+		(pts
 			(xy 151.13 91.44) (xy 161.29 91.44)
 		)
@@
 	(wire
 		(pts
+			(xy 34.29 121.92) (xy 34.29 104.14)
+		)
+		(stroke
+			(width 0)
+			(type default)
+		)
+	)
+	(wire
+		(pts
 			(xy 100.33 91.44) (xy 86.36 91.44)
 		)
@@
 	(wire
 		(pts
+			(xy 184.15 60.96) (xy 205.74 60.96)
+		)
+		(stroke
+			(width 0)
+			(type default)
+		)
+	)
+	(wire
+		(pts
 			(xy 177.8 82.55) (xy 184.15 82.55)
 		)
@@
 			(width 0)
 			(type solid)
+		)
+	)
+	(wire
+		(pts
+			(xy 208.28 121.92) (xy 208.28 123.19)
+		)
+		(stroke
+			(width 0)
+			(type default)
 		)
 	)
@@
 			(effects
 				(font
+					(size 1.27 1.27)
+				)
+				(justify left)
+				(hide yes)
+			)
+		)
+	)
+	(global_label "Boost Ground (V-)"
+		(shape input)
+		(at 208.28 123.19 0)
+		(fields_autoplaced yes)
+		(effects
+			(font
+				(size 1.27 1.27)
+				(bold yes)
+			)
+			(justify left)
+		)
+		(property "Intersheetrefs" "${INTERSHEET_REFS}"
+			(at 230.0048 123.19 0)
+			(effects
+				(font
+					(size 1.27 1.27)
+				)
+				(justify left)
+				(hide yes)
+			)
+		)
+	)
+	(global_label "Boost Output (Vout)"
+		(shape input)
+		(at 205.74 60.96 0)
+		(fields_autoplaced yes)
+		(effects
+			(font
+				(size 1.27 1.27)
+				(bold yes)
+			)
+			(justify left)
+		)
+		(property "Intersheetrefs" "${INTERSHEET_REFS}"
+			(at 228.4928 60.96 0)
+			(effects
+				(font
+					(size 1.27 1.27)
+				)
+				(justify left)
+				(hide yes)
+			)
+		)
+	)
+	(global_label "Battery Box Vin (Connectors)"
+		(shape input)
+		(at 34.29 104.14 90)
+		(fields_autoplaced yes)
+		(effects
+			(font
+				(size 1.27 1.27)
+				(bold yes)
+			)
+			(justify left)
+		)
+		(property "Intersheetrefs" "${INTERSHEET_REFS}"
+			(at 34.29 72.4971 90)
+			(effects
+				(font

Commit message: Add files via upload
Finished the main schematic as well as the sub schematics
Parts:
- removed U11: LM2735X, Boost Converter Chip:MF05A, symbol 2024-09-27_13-12-28-eagle-import:LM2735XMF/NOPBLM2735XMF/NOPB
- added U5: LM2735XMF/NOPB, Boost:MF05A, symbol Boost Chip:LM2735XMF_NOPB
Connections:
- net Battery Box Vout (Flyback Diode): now also U5.5 (VIN)
- net Earth: now also U5.2 (GND)
- net at C4.1, R2.1, R3.1: now also U5.3 (FB)
- net at D3.2 (A), L2.2: now also U5.1 (SW)
- net at R1.2: now also U5.4 (EN)
Other:
- moved on the sheet: R1
Changed lines of the file:
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@@
 	(paper "A4")
 	(junction
+		(at 95.25 121.92)
+		(diameter 0)
+		(color 0 0 0 0)
+	)
+	(junction
 		(at 125.73 121.92)
 		(diameter 0)
@@
 	(wire
 		(pts
+			(xy 154.94 88.9) (xy 151.13 88.9)
+		)
+		(stroke
+			(width 0)
+			(type default)
+		)
+	)
+	(wire
+		(pts
 			(xy 69.85 60.96) (xy 86.36 60.96)
 		)
@@
 	(wire
 		(pts
+			(xy 154.94 74.93) (xy 154.94 88.9)
+		)
+		(stroke
+			(width 0)
+			(type default)
+		)
+	)
+	(wire
+		(pts
 			(xy 151.13 91.44) (xy 161.29 91.44)
 		)
@@
 	(wire
 		(pts
-			(xy 100.33 91.44) (xy 86.36 91.44)
-		)
-		(stroke
-			(width 0)
-			(type default)
-		)
-	)
-	(wire
-		(pts
 			(xy 140.97 60.96) (xy 154.94 60.96)
 		)
@@
 	(wire
 		(pts
-			(xy 86.36 91.44) (xy 86.36 86.36)
-		)
-		(stroke
-			(width 0)
-			(type default)
-		)
-	)
-	(wire
-		(pts
 			(xy 69.85 60.96) (xy 69.85 95.25)
 		)
@@
 	(wire
 		(pts
+			(xy 95.25 88.9) (xy 95.25 121.92)
+		)
+		(stroke
+			(width 0)
+			(type default)
+		)
+	)
+	(wire
+		(pts
 			(xy 69.85 102.87) (xy 69.85 121.92)
 		)
@@
 	(wire
 		(pts
+			(xy 151.13 86.36) (xy 151.13 80.01)
+		)
+		(stroke
+			(width 0)
+			(type default)
+		)
+	)
+	(wire
+		(pts
 			(xy 177.8 82.55) (xy 184.15 82.55)
 		)
@@
 	(wire
 		(pts
-			(xy 125.73 106.68) (xy 125.73 121.92)
+			(xy 95.25 121.92) (xy 125.73 121.92)
+		)
+		(stroke
+			(width 0)
+			(type default)
+		)
+	)
+	(wire
+		(pts
+			(xy 151.13 80.01) (xy 110.49 80.01)
 		)
 		(stroke
@@
 	(wire
 		(pts
-			(xy 86.36 78.74) (xy 86.36 60.96)
-		)
-		(stroke
-			(width 0)
-			(type default)
-		)
-	)
-	(wire
-		(pts
-			(xy 69.85 121.92) (xy 125.73 121.92)
+			(xy 86.36 67.31) (xy 86.36 60.96)
+		)
+		(stroke
+			(width 0)
+			(type default)
+		)
+	)
+	(wire
+		(pts
+			(xy 69.85 121.92) (xy 95.25 121.92)
 		)
 		(stroke
@@
 	(wire
 		(pts
+			(xy 95.25 86.36) (xy 95.25 76.2)
+		)
+		(stroke
+			(width 0)
+			(type default)
+		)
+	)
+	(wire
+		(pts
 			(xy 161.29 82.55) (xy 161.29 91.44)
 		)
@@
 	(wire
 		(pts
-			(xy 110.49 76.2) (xy 110.49 60.96)
+			(xy 110.49 60.96) (xy 110.49 80.01)
 		)
 		(stroke
@@
 	(wire
 		(pts
+			(xy 95.25 76.2) (xy 140.97 76.2)
+		)
+		(stroke
+			(width 0)
+			(type default)
+		)
+	)
+	(wire
+		(pts
 			(xy 34.29 60.96) (xy 34.29 57.15)
+		)
+		(stroke
+			(width 0)
+			(type default)
+		)
+	)
+	(wire
+		(pts
+			(xy 86.36 74.93) (xy 154.94 74.93)
 		)
 		(stroke
@@
 	)
 	(symbol
-		(lib_id "2024-09-27_13-12-28-eagle-import:LM2735XMF/NOPBLM2735XMF/NOPB")
-		(at 125.73 91.44 0)
-		(unit 1)
-		(exclude_from_sim no)
-		(in_bom yes)
-		(on_board yes)
-		(dnp no)
-		(property "Reference" "U11"
-			(at 125.73 91.44 0)
-			(effects
-				(font
-					(size 2 1.7)
-				)
-				(justify bottom)
-				(hide yes)
-			)
-		)
-		(property "Value" "LM2735X"
-			(at 125.73 95.25 0)
-			(effects
-				(font
-					(size 2 1.7)
-				)
-				(justify bottom)
-			)
-		)
-		(property "Footprint" "Boost Converter Chip:MF05A"
-			(at 125.73 91.44 0)
-			(effects
-				(font
-					(size 1.27 1.27)
-				)
-				(hide yes)
-			)
-		)
-		(property "Datasheet" ""
-			(at 125.73 91.44 0)
-			(effects
-				(font
-					(size 1.27 1.27)
-				)
-				(hide yes)
-			)
-		)
-		(property "Description" ""
-			(at 125.73 91.44 0)
-			(effects
-				(font
-					(size 1.27 1.27)
-				)
-				(hide yes)
-			)
-		)
-		(pin "1"
-		)
-		(pin "2"
-		)
-		(pin "3"
-		)
-		(pin "4"
-		)
-		(pin "5"
-		)
-		(instances
-			(project "PCB desing"
-				(path "/eb9a8801-b205-4599-90e8-b0089b4de1f9/75f61d54-82fa-43c7-a51b-df767089e132"
-					(reference "U11")
-					(unit 1)
-				)
-			)
-		)
-	)
-	(symbol
 		(lib_id "Device:R_US")
 		(at 172.72 69.85 90)
@@
 	)
 	(symbol
-		(lib_id "Device:R_US")
-		(at 86.36 82.55 0)
+		(lib_id "Boost Chip:LM2735XMF_NOPB")
+		(at 95.25 86.36 0)
 		(unit 1)
 		(exclude_from_sim no)
@@
 		(dnp no)
 		(fields_autoplaced yes)
+		(property "Reference" "U5"
+			(at 123.19 76.2 0)
+			(effects
+				(font
+					(size 1.524 1.524)
+				)
+			)
+		)
+		(property "Value" "LM2735XMF/NOPB"
+			(at 123.19 78.74 0)
+			(effects
+				(font
+					(size 1.524 1.524)
+				)
+			)
+		)
+		(property "Footprint" "Boost:MF05A"
+			(at 95.25 86.36 0)
+			(effects
+				(font
+					(size 1.27 1.27)
+					(italic yes)
+				)
+				(hide yes)
+			)
+		)
+		(property "Datasheet" "LM2735XMF/NOPB"
+			(at 95.25 86.36 0)
+			(effects
+				(font
+					(size 1.27 1.27)
+					(italic yes)
+				)
+				(hide yes)
+			)
+		)
+		(property "Description" ""
+			(at 95.25 86.36 0)
+			(effects
+				(font
+					(size 1.27 1.27)
+				)
+				(hide yes)
+			)
+		)
+		(pin "4"
+		)
+		(pin "3"
+		)
+		(pin "5"
+		)
+		(pin "1"
+		)
+		(pin "2"
+		)
+		(instances
+			(project "PCB desing"
+				(path "/eb9a8801-b205-4599-90e8-b0089b4de1f9/75f61d54-82fa-43c7-a51b-df767089e132"
+					(reference "U5")
+					(unit 1)
+				)
+			)
+		)
+	)
+	(symbol
+		(lib_id "Device:R_US")
+		(at 86.36 71.12 0)
+		(unit 1)
+		(exclude_from_sim no)
+		(in_bom yes)
+		(on_board yes)
+		(dnp no)
+		(fields_autoplaced yes)
 		(property "Reference" "R1"
-			(at 88.9 81.2799 0)
+			(at 88.9 69.8499 0)
 			(effects
 				(font
@@
 		)
 		(property "Value" "10k Ohms"
-			(at 88.9 83.8199 0)
+			(at 88.9 72.3899 0)
 			(effects
 				(font
@@
 		)
 		(property "Footprint" ""
-			(at 87.376 82.804 90)
+			(at 87.376 71.374 90)
 			(effects
 				(font
@@
 		)
 		(property "Datasheet" "~"
-			(at 86.36 82.55 0)
+			(at 86.36 71.12 0)
 			(effects
 				(font
@@
 		)
 		(property "Description" ""
-			(at 86.36 82.55 0)
-			(effects
-				(font
+			(at 86.36 71.12 0)
+			(effects
+				(font
