File: Power_amp.kicad_sch (KiCad schematic)
At the start: 0 parts

Commit message: Add files via upload
Finished everything except for the micro schematic
Parts:
- added C10: 5V, symbol Device:C_Polarized_Small_US
- added C11: .1 uF, symbol Device:C
- added C12: 100 uF, symbol Device:C
- added C6: 100 uF, symbol Device:C_Polarized_Small_US
- added C7, C8: .1 uF, symbol Device:C_Polarized_Small_US
- added C9: 1000 uF, symbol Device:C_Polarized_Small_US
- added J3: Conn_01x02_Pin, symbol Connector:Conn_01x02_Pin
- added J4: Conn_01x02_Socket, symbol Connector:Conn_01x02_Socket
- added U8: LM386, symbol Amplifier_Audio:LM386
Connections:
- new net: C8.1, C9.1, U8.5
- new net: C7.1, U8.2 (-)
- new net: C9.2, J3.2 (Pin_2)
- new net: C11.2, U8.3 (+)
- new net: C6.1, U8.7 (BYPASS)
- new net Boost Output (Vout): U8.6 (V+)
- new net Connection to Speaker (V+): J4.2 (Pin_2)
- new net Connection to Speaker (V-): J4.1 (Pin_1)
- new net Earth: C10.2, C12.1, C6.2, C7.2, C8.2, J3.1 (Pin_1), U8.4 (GND)
- new net Micro DAC PA4 (Pin 20): C11.1
- new net VCC: C10.1, C12.2
- no-connect marks 0 -> 2
