File: PCB/Schematic/PCB/PCB.kicad_pcb (KiCad board)
At the start: 2 copper layers, 5 parts, among them U1 STM32L476RGTx, U2 FGPMMOPA6H, U4 TPS63001DRC, U5 LM2735X

Commit message: Add files via upload
Parts:
- added C1: 10 uF, 1mOhms, Capacitor_SMD:C_0805_2012Metric, F.Cu at (81.3, 128.0)
- added C11: .1 uF, Capacitor_SMD:C_0805_2012Metric, F.Cu at (177.8, 160.0)
- added C2: 47 uF, 2.94 mOhms, Capacitor_SMD:C_0805_2012Metric, F.Cu at (106.7, 130.5)
- added C3: 10 uF, 3 mOhms, Resistor_SMD:R_0805_2012Metric, F.Cu at (83.8, 171.1)
- added C4: 1.8 nF, Capacitor_SMD:C_0805_2012Metric, F.Cu at (95.6, 175.3)
- added C5: 22 uF, 1 mOhms, Resistor_SMD:R_0805_2012Metric, F.Cu at (88.9, 180.3)
- added C6: 100 uF, Polarized Caps (.1 - 100 uF):CAP_UZE_4X3P9_NCH, F.Cu at (190.5, 172.7)
- added C7: .1 uF, Polarized Caps (.1 - 100 uF):CAP_UZE_4X3P9_NCH, F.Cu at (173.4, 175.3)
- added C8: .1 uF, Polarized Caps (.1 - 100 uF):CAP_UZE_4X3P9_NCH, F.Cu at (195.6, 172.7)
- added C9: 1000 uF, Polarized Cap 1000 uF:PCAP_10x10-ELECT_NCA, F.Cu at (223.5, 157.5)
- added D1: D, Schottky:Schottky, F.Cu at (55.9, 172.7)
- added D3: 320 mV, 2A, Schottky:Schottky, F.Cu at (135.0, 177.8)
- added FB2: FerriteBead, Ferrite_THT:LairdTech_28C0236-0JW-10, F.Cu at (94.0, 61.0)
- added FB3: FerriteBead, Ferrite_THT:LairdTech_28C0236-0JW-10, F.Cu at (101.6, 68.6)
- added J2: Conn_01x02_Pin, Connector_JST:JST_PH_B2B-PH-SM4-TB_1x02-1MP_P2.00mm_Vertical, F.Cu at (39.6, 182.4)
- added J3: Conn_01x02_Pin, Connector_JST:JST_PH_B2B-PH-SM4-TB_1x02-1MP_P2.00mm_Vertical, F.Cu at (278.9, 158.5)
- added L1: 3.3 uH, 20 mOhms, Inductor_SMD:L_0805_2012Metric, F.Cu at (82.8, 119.4)
- added L2: 3.3 uH, 20 Ohm, Inductor_SMD:L_TDK_SLF7045, F.Cu at (123.8, 175.3)
- added R1: 10k Ohms, Resistor_SMD:R_0805_2012Metric, F.Cu at (111.8, 171.8)
- added R2: 10k Ohms, Resistor_SMD:R_0805_2012Metric, F.Cu at (101.6, 179.4)
- added R3: 30k Ohms, Resistor_SMD:R_0805_2012Metric, F.Cu at (95.6, 180.3)
- added U8: LM386, LM386:LM386, F.Cu at (187.8, 158.1)
- moved U2 107.3 mm to (35.2, 96.3), turned to 180 degrees
- moved U5 81.6 mm to (102.9, 171.8)
- moved U3 76.7 mm to (170.2, 66.0), turned to 0 degrees
- moved U4 35.3 mm to (94.0, 125.4)
- moved U1 28.4 mm to (116.2, 51.1)
Connections:
- U1 pad 10: unconnected-(U1-PC2-Pad10) -> (no net)
- U1 pad 11: unconnected-(U1-PC3-Pad11) -> (no net)
- U1 pad 14: Net-(U1-PA0) -> (no net)
- U1 pad 15: Net-(U1-PA1) -> (no net)
- U1 pad 16: unconnected-(U1-PA2-Pad16) -> (no net)
- U1 pad 17: unconnected-(U1-PA3-Pad17) -> (no net)
- U1 pad 2: unconnected-(U1-PC13-Pad2) -> (no net)
- U1 pad 20: Net-(U1-PA4) -> (no net)
- U1 pad 21: unconnected-(U1-PA5-Pad21) -> (no net)
- U1 pad 22: unconnected-(U1-PA6-Pad22) -> (no net)
- U1 pad 23: unconnected-(U1-PA7-Pad23) -> (no net)
- U1 pad 24: unconnected-(U1-PC4-Pad24) -> (no net)
- U1 pad 25: unconnected-(U1-PC5-Pad25) -> (no net)
- U1 pad 26: unconnected-(U1-PB0-Pad26) -> (no net)
- U1 pad 27: unconnected-(U1-PB1-Pad27) -> (no net)
- U1 pad 28: unconnected-(U1-PB2-Pad28) -> (no net)
- U1 pad 29: unconnected-(U1-PB10-Pad29) -> (no net)
- U1 pad 3: unconnected-(U1-PC14-Pad3) -> (no net)
- U1 pad 30: unconnected-(U1-PB11-Pad30) -> (no net)
- U1 pad 33: unconnected-(U1-PB12-Pad33) -> (no net)
- U1 pad 34: unconnected-(U1-PB13-Pad34) -> (no net)
- U1 pad 35: unconnected-(U1-PB14-Pad35) -> (no net)
- U1 pad 36: unconnected-(U1-PB15-Pad36) -> (no net)
- U1 pad 37: unconnected-(U1-PC6-Pad37) -> (no net)
- U1 pad 38: unconnected-(U1-PC7-Pad38) -> (no net)
- U1 pad 39: unconnected-(U1-PC8-Pad39) -> (no net)
- U1 pad 4: unconnected-(U1-PC15-Pad4) -> (no net)
- U1 pad 40: unconnected-(U1-PC9-Pad40) -> (no net)
- U1 pad 41: unconnected-(U1-PA8-Pad41) -> (no net)
- U1 pad 42: unconnected-(U1-PA9-Pad42) -> (no net)
- U1 pad 43: unconnected-(U1-PA10-Pad43) -> (no net)
- U1 pad 44: unconnected-(U1-PA11-Pad44) -> (no net)
- U1 pad 45: unconnected-(U1-PA12-Pad45) -> (no net)
- U1 pad 46: unconnected-(U1-PA13-Pad46) -> (no net)
- U1 pad 49: unconnected-(U1-PA14-Pad49) -> (no net)
- U1 pad 5: unconnected-(U1-PH0-Pad5) -> (no net)
- U1 pad 50: unconnected-(U1-PA15-Pad50) -> (no net)
- U1 pad 51: unconnected-(U1-PC10-Pad51) -> (no net)
- U1 pad 52: unconnected-(U1-PC11-Pad52) -> (no net)
- U1 pad 53: Net-(U1-PC12) -> (no net)
- U1 pad 54: Net-(U1-PD2) -> (no net)
- U1 pad 55: unconnected-(U1-PB3-Pad55) -> (no net)
- U1 pad 56: unconnected-(U1-PB4-Pad56) -> (no net)
- U1 pad 57: unconnected-(U1-PB5-Pad57) -> (no net)
- U1 pad 58: unconnected-(U1-PB6-Pad58) -> (no net)
- U1 pad 59: unconnected-(U1-PB7-Pad59) -> (no net)
- U1 pad 6: unconnected-(U1-PH1-Pad6) -> (no net)
- U1 pad 60: unconnected-(U1-BOOT0-Pad60) -> (no net)
- U1 pad 61: unconnected-(U1-PB8-Pad61) -> (no net)
- U1 pad 62: unconnected-(U1-PB9-Pad62) -> (no net)
- U1 pad 7: unconnected-(U1-NRST-Pad7) -> (no net)
- U1 pad 8: unconnected-(U1-PC0-Pad8) -> (no net)
- U1 pad 9: unconnected-(U1-PC1-Pad9) -> (no net)
- U2 pad P$10: Net-(U1-PA0) -> (no net)
- U2 pad P$11: unconnected-(U2-EX_ANT-PadP$11) -> (no net)
- U2 pad P$13: unconnected-(U2-1PPS-PadP$13) -> (no net)
- U2 pad P$14: unconnected-(U2-RTCM-PadP$14) -> (no net)
- U2 pad P$15: unconnected-(U2-NC@3-PadP$15) -> (no net)
- U2 pad P$16: unconnected-(U2-NC@4-PadP$16) -> (no net)
- U2 pad P$17: unconnected-(U2-NC@5-PadP$17) -> (no net)
- U2 pad P$18: unconnected-(U2-NC@6-PadP$18) -> (no net)
- U2 pad P$2: unconnected-(U2-NRESET-PadP$2) -> (no net)
- U2 pad P$20: unconnected-(U2-NC@7-PadP$20) -> (no net)
- U2 pad P$5: unconnected-(U2-3D-FIX-PadP$5) -> (no net)
- U2 pad P$6: unconnected-(U2-NC@1-PadP$6) -> (no net)
- U2 pad P$7: unconnected-(U2-NC@2-PadP$7) -> (no net)
- U2 pad P$9: Net-(U1-PA1) -> (no net)
- U3 pad 3: Net-(U1-PC12) -> (no net)
- U3 pad 4: Net-(U1-PD2) -> (no net)
- U3 pad 5: unconnected-(U3-NC-Pad5) -> (no net)
- U4 pad 2: Net-(U4-L2@2) -> (no net)
- U4 pad 4: Net-(U4-L1@4) -> (no net)
Routing:
- net PAD: track 0.00 -> 976.6 mm, vias 0 -> 3
- net (no net): track 0.00 -> 453.7 mm, vias 0 -> 8
- net Net-(U1-VBAT): track 0.00 -> 369.2 mm
- net Net-(J2-Pin_2): track 0.00 -> 196.3 mm, vias 0 -> 2
- net Net-(D3-K): track 0.00 -> 161.9 mm, vias 0 -> 4
- net Net-(D3-A): track 0.00 -> 56.5 mm, vias 0 -> 2
- net Net-(J3-Pin_2): track 0.00 -> 51.7 mm
- net Net-(C8-Pad1): track 0.00 -> 40.8 mm
- net Net-(D1-K): track 0.00 -> 30.0 mm
- net Net-(D1-A): track 0.00 -> 23.9 mm
- net Net-(U8--): track 0.00 -> 22.7 mm, vias 0 -> 2
- net Net-(U5-FB@4): track 0.00 -> 21.9 mm
- net Net-(U1-VDDA): track 0.00 -> 19.1 mm
- net Net-(U1-VSSA): track 0.00 -> 17.8 mm
- net Net-(U8-BYPASS): track 0.00 -> 17.0 mm, vias 0 -> 2
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Other:
- board text added: "AMP"
