File: Hierarchy PCB/Boost.kicad_sch (KiCad schematic)
At the start: 9 parts, among them U11 LM2735X

Commit message: Add files via upload
Parts:
- removed U11: LM2735X, Boost Converter Chip:MF05A, symbol 2024-09-27_13-12-28-eagle-import:LM2735XMF/NOPBLM2735XMF/NOPB
- added U5: LM2735XMF/NOPB, Boost:MF05A, symbol Boost Chip:LM2735XMF_NOPB
Connections:
- net Battery Box Vout (Flyback Diode): now also U5.5 (VIN)
- net Earth: now also U5.2 (GND)
- net at C4.1, R2.1, R3.1: now also U5.3 (FB)
- net Boost Output (Vout): now reaches C4.2, C5.1, D3.1 (K), R3.2
- net at D3.2 (A), L2.2: now also U5.1 (SW)
- net at R1.2: now also U5.4 (EN)
Other:
- moved on the sheet: R1
