File: Hierarchy PCB/Buck_Boost.kicad_sch (KiCad schematic)
At the start: 4 parts, among them U7 TPS63001DRC

Commit message: Add files via upload
Parts:
- removed U7: TPS63001DRC, Buck-Boost Converter Chip:DRC0010J, symbol 2024-09-27_13-12-33-eagle-import:TPS63001DRCRTPS63001DRCR
- added U7: TPS63001DRCR, Buck-Boost:DRC0010J, symbol Buck-Boost Chip:TPS63001DRCR
Connections:
- net Earth: now also U7.11 (PAD), U7.3 (PGND), U7.9 (GND)
- net GPS Pin Four (Vbackup): no longer C2.1
- net at L3.2: now also U7.2 (L2)
- net at L3.1: now also U7.4 (L1)
- net Battery Box Vout (Flyback Diode) renamed Battery Box Voltage
- net Battery Box Voltage: now also U7.5 (VIN), U7.6 (EN), U7.7 (PS_SYNC), U7.8 (VINA)
- new net Buck-Boost Voltage: C2.1, U7.1 (VOUT), U7.10 (FB)
