File: Hierarchy PCB/GPS.kicad_sch (KiCad schematic)
At the start: 1 part, among them U10 FGPMMOPA6H

Commit message: Add files via upload
Connections:
- net Buck Boost Pin One (Vout) renamed Buck-Boost Voltage
- net Micro UART RX PA1 (Pin 15) renamed Micro GPS RX
- net Micro UART TX PA0 (Pin 14) renamed Micro GPS TX
Changed lines of the file:
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@@
 		(color 0 0 0 0)
 	)
+	(junction
+		(at 160.02 88.9)
+		(diameter 0)
+		(color 0 0 0 0)
+	)
 	(wire
 		(pts
@@
 		(pts
 			(xy 72.39 104.14) (xy 72.39 135.89)
+		)
+		(stroke
+			(width 0)
+			(type default)
+		)
+	)
+	(wire
+		(pts
+			(xy 160.02 78.74) (xy 160.02 88.9)
 		)
 		(stroke
@@
 		)
 	)
-	(global_label "Micro UART RX PA1 (Pin 15)"
+	(global_label "Micro GPS RX"
 		(shape input)
 		(at 107.95 106.68 180)
@@
 		)
 		(property "Intersheetrefs" "${INTERSHEET_REFS}"
-			(at 76.7303 106.68 0)
+			(at 91.2446 106.68 0)
 			(effects
 				(font
@@
 		)
 	)
-	(global_label "Buck Boost Pin One (Vout)"
+	(global_label "GND"
+		(shape input)
+		(at 160.02 78.74 0)
+		(fields_autoplaced yes)
+		(effects
+			(font
+				(size 1.27 1.27)
+				(bold yes)
+			)
+			(justify left)
+		)
+		(property "Intersheetrefs" "${INTERSHEET_REFS}"
+			(at 167.3517 78.74 0)
+			(effects
+				(font
+					(size 1.27 1.27)
+				)
+				(justify left)
+				(hide yes)
+			)
+		)
+	)
+	(global_label "Buck-Boost Voltage"
 		(shape input)
 		(at 101.6 80.01 180)
@@
 		)
 		(property "Intersheetrefs" "${INTERSHEET_REFS}"
-			(at 72.0133 80.01 0)
+			(at 78.7262 80.01 0)
 			(effects
 				(font
@@
 		)
 	)
-	(global_label "Micro UART TX PA0 (Pin 14)"
+	(global_label "Micro GPS TX"
 		(shape input)
 		(at 107.95 111.76 180)
@@
 		)
 		(property "Intersheetrefs" "${INTERSHEET_REFS}"
-			(at 77.0327 111.76 0)
-			(effects
-				(font
+			(at 91.547 111.76 0)
+			(effects
+				(font
