File: Hierarchy PCB/untitled.kicad_sch (KiCad schematic)
At the start: 1 part

Commit message: Add files via upload
Connections:
- net Micro (PC12) renamed Micro LoRa TX
- net Micro (PD2) renamed Micro LoRa RX
- net U4 Pin (Vout) renamed Buck-Boost Voltage
Changed lines of the file:
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@@
 		)
 	)
-	(global_label "Micro (PD2)"
+	(global_label "Micro LoRa RX"
 		(shape input)
 		(at 140.97 130.81 270)
@@
 		)
 		(property "Intersheetrefs" "${INTERSHEET_REFS}"
-			(at 140.97 145.2857 90)
+			(at 140.97 147.886 90)
 			(effects
 				(font
@@
 		)
 	)
-	(global_label "Micro (PC12)"
+	(global_label "Micro LoRa TX"
 		(shape input)
 		(at 135.89 130.81 270)
@@
 		)
 		(property "Intersheetrefs" "${INTERSHEET_REFS}"
-			(at 135.89 146.4952 90)
+			(at 135.89 147.5836 90)
 			(effects
 				(font
@@
 		)
 	)
-	(global_label "U4 Pin (Vout)"
+	(global_label "Buck-Boost Voltage"
 		(shape input)
 		(at 130.81 130.81 270)
@@
 		)
 		(property "Intersheetrefs" "${INTERSHEET_REFS}"
-			(at 130.81 147.0999 90)
+			(at 130.81 153.2078 90)
 			(effects
 				(font
@@
 		)
 	)
-	(global_label "U4 Pin (Vout)"
+	(global_label "Buck-Boost Voltage"
 		(shape input)
 		(at 125.73 130.81 270)
@@
 		)
 		(property "Intersheetrefs" "${INTERSHEET_REFS}"
-			(at 125.73 147.0999 90)
+			(at 125.73 153.2078 90)
 			(effects
 				(font
