File: PCB/_autosave-PCB.kicad_sch (KiCad schematic)
At the start: 50 parts, among them J1 Conn_01x02_Socket, J2 Conn_01x02_Pin, J3 Conn_01x02_Pin, J4 Conn_01x02_Socket, J5 Programming Pin, J6 Programming Pin, J7 Programming Pin, J8 Programming Pin, U1 STM32L476RGTx, U2 FGPMMOPA6H, U4 TPS63001DRCR, U5 LM2735XMF/NOPB, U8 LM386, U9 MAX7375AXR805

Commit message: Add files via upload
Parts:
- removed FB1, FB4: FerriteBead, Ferrite_THT:LairdTech_28C0236-0JW-10, symbol Device:FerriteBead
- added C18: .1 uF, Capacitor_SMD:C_0805_2012Metric_Pad1.18x1.45mm_HandSolder, symbol Device:C
- added R4, R5: 0 Ohms, Resistor_SMD:R_0805_2012Metric_Pad1.20x1.40mm_HandSolder, symbol Device:R_US
- D1: value D -> 320 mV, 2A
Connections:
- net GND is gone; now on net Earth: C10.1, C10.2, C13.1, C13.2, C14.1, C14.2, C15.1, C15.2, C19.1, C2.1, U1.1 (VBAT), U1.19 (VDD), U1.32 (VDD), U1.48 (VDDUSB), U1.64 (VDD), U2.P$1 (VCC), U2.P$4 (VBACKUP), U3.1 (VDD), U3.2 (NRST), U4.1 (VOUT), U4.10 (FB), U9.1 (V+)
- net Earth: now also C18.1, C18.2, R4.1, R5.1; no longer U1.12 (VSSA)
- net VDDA Connection: now also R4.2
- net at C11.1, U1.20 (PA4): no longer U1.15 (PA1), U2.P$9 (TX)
- net at U1.14 (PA0): no longer U2.P$10 (RX)
- net at U1.42 (PA9): now also U2.P$10 (RX)
- net at U1.43 (PA10): now also U2.P$9 (TX)
- net VDDA GND Connection: now reaches C16.2, C17.2
- net VDDA GND Connection: now also U1.12 (VSSA), R5.2
