File: PCB/PCB.kicad_pcb (KiCad board)
At the start: 2 copper layers, 36 parts, among them J2 Conn_01x02_Pin, J3 Conn_01x02_Pin, U1 STM32L476RGTx, U2 FGPMMOPA6H, U4 TPS63001DRCR, U5 LM2735XMF/NOPB, U8 LM386, U9 MAX7375AXR805

Commit message: Add files via upload
Parts:
- C10, C13, C14, C15, C16, C17, FB1, FB4: moved to B.Cu
- moved J2 112.6 mm to (108.2, 99.0)
- moved D1 95.7 mm to (114.3, 89.3), turned to -90 degrees
- moved U5 76.4 mm to (135.8, 89.9)
- moved C3 74.2 mm to (121.9, 88.9), turned to -90 degrees
- moved L1 56.7 mm to (112.3, 81.7), turned to 90 degrees
- moved U3 56.4 mm to (185.4, 53.3)
- moved C4 56.4 mm to (143.7, 104.1)
- moved R1 56.4 mm to (141.3, 113.9)
- moved C5 56.4 mm to (143.7, 107.2)
- moved L2 56.4 mm to (152.4, 116.8)
- moved R2 56.4 mm to (141.3, 116.8)
- moved D3 56.4 mm to (162.6, 111.8)
- moved R3 56.4 mm to (141.3, 119.8)
- moved C2 54.8 mm to (119.6, 77.4), turned to 180 degrees
- moved FB4 49.6 mm to (121.9, 68.6)
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Connections:
- C1 pad 2: PAD -> Buck-Boost Voltage
- C12 pad 2: PAD -> Buck-Boost Voltage
- C16 pad 2: Net-(C16-Pad2) -> VDDA GND Connection
- C17 pad 2: Net-(C16-Pad2) -> VDDA GND Connection
- C19 pad 2: PAD -> Buck-Boost Voltage
- C2 pad 2: PAD -> Buck-Boost Voltage
- C3 pad 2: PAD -> Buck-Boost Voltage
- C5 pad 2: PAD -> Buck-Boost Voltage
- C6 pad 2: PAD -> Buck-Boost Voltage
- C7 pad 2: PAD -> Buck-Boost Voltage
- C8 pad 2: PAD -> Buck-Boost Voltage
- FB4 pad 2: Net-(C16-Pad2) -> VDDA GND Connection
- J2 pad 1: PAD -> Buck-Boost Voltage
- J3 pad 1: PAD -> Buck-Boost Voltage
- R2 pad 2: PAD -> Buck-Boost Voltage
- U1 pad 12: PAD -> VDDA GND Connection
- U1 pad 18: PAD -> Buck-Boost Voltage
- U1 pad 31: PAD -> Buck-Boost Voltage
- U1 pad 47: PAD -> Buck-Boost Voltage
- U1 pad 63: PAD -> Buck-Boost Voltage
- U2 pad P$12: PAD -> Buck-Boost Voltage
- U2 pad P$19: PAD -> Buck-Boost Voltage
- U2 pad P$3: PAD -> Buck-Boost Voltage
- U2 pad P$8: PAD -> Buck-Boost Voltage
- U3 pad 6: PAD -> Buck-Boost Voltage
- U4 pad 11: PAD -> Buck-Boost Voltage
- U4 pad 3: PAD -> Buck-Boost Voltage
- U4 pad 9: PAD -> Buck-Boost Voltage
- U5 pad 2: PAD -> Buck-Boost Voltage
- U8 pad 4: PAD -> Buck-Boost Voltage
- U9 pad 3: PAD -> Buck-Boost Voltage
Routing:
- net Buck-Boost Voltage: track 11.0 -> 237.6 mm, vias 0 -> 17
- net PAD: track 104.3 -> 0.00 mm
- net Net-(D1-K): track 75.8 -> 24.1 mm
- net Net-(D1-A): track 30.9 -> 10.1 mm
- net VDDA GND Connection: track 0.00 -> 12.9 mm, vias 0 -> 1
- net VDDA Connection: track 0.00 -> 11.3 mm, vias 0 -> 1
- net Net-(U4-L2): track 0.00 -> 4.71 mm
- net Net-(U4-L1): track 0.00 -> 4.45 mm
- net Net-(U1-PH0): track 5.67 -> 3.90 mm

Commit message: Add files via upload
Need to decide how big the ground plane is, where to place the GPS, and connect the LoRa and GPS traces.
Also need to add silkscreen layer and make sure checks in PCB verification checklist are completed.
Parts:
- added C18: .1 uF, Capacitor_SMD:C_0805_2012Metric_Pad1.18x1.45mm_HandSolder, F.Cu at (147.7, 73.2)
- D1: value D -> 320 mV, 2A
- moved U2 156.2 mm to (187.6, 68.8)
- moved J3 96.3 mm to (190.3, 109.8)
- moved C7 72.0 mm to (152.9, 113.2), turned to -90 degrees
- moved C6 64.7 mm to (159.1, 113.2), turned to -90 degrees
- moved C8 61.9 mm to (165.4, 113.3), turned to -90 degrees
- moved U3 56.9 mm to (129.9, 65.6), turned to 90 degrees
- moved U8 51.4 mm to (162.1, 106.1)
- moved C11 50.3 mm to (154.5, 105.8), turned to -90 degrees
- moved C12 38.3 mm to (168.7, 104.2), turned to -90 degrees
- moved C9 32.1 mm to (176.9, 108.8)
- moved U5 20.3 mm to (146.3, 107.2)
- moved L2 19.9 mm to (137.5, 103.7)
- moved C2 19.1 mm to (127.5, 94.7)
- moved L1 19.1 mm to (120.3, 99.1)
- moved U4 19.1 mm to (125.9, 99.6)
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Connections:
- C11 pad 1: Net-(U1-PA1) -> Net-(U1-PA4)
- U1 pad 20: Net-(U1-PA1) -> Net-(U1-PA4)
Routing:
- net Buck-Boost Voltage: track 237.6 -> 385.8 mm, vias 17 -> 21
- net Net-(D3-K): track 0.00 -> 51.2 mm, vias 0 -> 2
- net Net-(D1-K): track 24.1 -> 68.9 mm, vias 0 -> 2
- net Net-(U1-PA4): track 0.00 -> 27.8 mm
- net Net-(U5-FB): track 0.00 -> 21.0 mm
- net Net-(C8-Pad1): track 0.00 -> 11.3 mm
- net Net-(U8--): track 0.00 -> 9.89 mm, vias 0 -> 2
- net Net-(J3-Pin_2): track 0.00 -> 9.75 mm
- net Net-(U8-BYPASS): track 0.00 -> 8.53 mm
- net Net-(U5-EN): track 0.00 -> 6.01 mm
- net Net-(U8-+): track 0.00 -> 4.94 mm
- net Net-(J7-Pin_1): track 0.00 -> 2.58 mm, vias 0 -> 1
- net Net-(J6-Pin_1): track 0.00 -> 2.12 mm, vias 0 -> 1
- net Net-(J8-Pin_1): track 0.00 -> 1.95 mm, vias 0 -> 1
- net Net-(J5-Pin_1): track 0.00 -> 1.70 mm, vias 0 -> 1
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- added copper zone on B.Cu, net VDDA GND Connection
- added copper zone on F.Cu, net VDDA GND Connection

Commit message: Add files via upload
Parts:
- removed FB1, FB4: FerriteBead, Ferrite_THT:LairdTech_28C0236-0JW-10
- added R4: 0 Ohms, Resistor_SMD:R_0805_2012Metric_Pad1.20x1.40mm_HandSolder, B.Cu at (123.9, 89.7)
- added R5: 0 Ohms, Resistor_SMD:R_0805_2012Metric_Pad1.20x1.40mm_HandSolder, B.Cu at (120.8, 82.1)
- added REF**: MountingHole_2.2mm_M2, MountingHole:MountingHole_2.2mm_M2, F.Cu at (190.5, 114.3)
- added REF**: MountingHole_2.2mm_M2, MountingHole:MountingHole_2.2mm_M2, F.Cu at (190.5, 71.3)
- added REF**: MountingHole_2.2mm_M2, MountingHole:MountingHole_2.2mm_M2, F.Cu at (92.2, 116.5)
- added REF**: MountingHole_2.2mm_M2, MountingHole:MountingHole_2.2mm_M2, F.Cu at (92.4, 71.1)
- C18: moved to B.Cu
- moved U3 36.6 mm to (101.6, 88.9), turned to 180 degrees
- moved U2 20.0 mm to (175.0, 84.2)
- moved C18 10.8 mm to (154.9, 81.3)
- moved J3 6.67 mm to (190.3, 103.1)
Connections:
- U1 pad 14: Net-(U1-PA0) -> unconnected-(U1-PA0-Pad14)
- U1 pad 15: Net-(U1-PA1) -> unconnected-(U1-PA1-Pad15)
- U1 pad 42: unconnected-(U1-PA9-Pad42) -> Net-(U1-PA9)
- U1 pad 43: unconnected-(U1-PA10-Pad43) -> Net-(U1-PA10)
- U2 pad P$10: Net-(U1-PA0) -> Net-(U1-PA9)
- U2 pad P$9: Net-(U1-PA1) -> Net-(U1-PA10)
Routing:
- net Buck-Boost Voltage: track 385.8 -> 579.8 mm, vias 21 -> 27
- net Net-(U1-PD2): track 0.00 -> 47.9 mm
- net Net-(U1-PC12): track 0.00 -> 44.8 mm, vias 0 -> 1
- net Net-(U1-PA9): track 0.00 -> 24.2 mm
- net Net-(U1-PA10): track 0.00 -> 23.8 mm
- net Net-(J3-Pin_2): track 9.75 -> 13.6 mm
- net Net-(U8--): track 9.89 -> 11.3 mm
- net VDDA GND Connection: track 12.9 -> 14.3 mm, vias 145 -> 35
- net Net-(D1-K): track 68.9 -> 69.9 mm
- net Net-(U5-EN): track 6.01 -> 6.80 mm
Other:
- board outline added: 105.5 x 51.8 mm
- board text added: "Connectors"
- board text added: "ECE 477 Team 5: Smart Dog Collar Andrew Wu David Manojlovic Nick Durnil Ethan James Revision: Version 1"
- board text added: "GPS Signal Connections (TX & RX)"
- board text added: "LM2735 Boost Chip"
- board text added: "LM386 Amplifier Chip"
- board text added: "LoRa Signal Connections (TX & RX)"
- board text added: "MTK MT3339 GPS Chip"
- board text added: "Pin 1"
- board text added: "RYLR896 LoRa Chip"
- board text added: "STM32L4"
- board text added: "TPS63 Buck-Boost Chip"

Commit message: changed pcb
Parts:
- added C20: .1 uF, Capacitor_SMD:C_0805_2012Metric_Pad1.18x1.45mm_HandSolder, F.Cu at (143.0, 71.0)
- added D2: LED, LED_SMD:LED_0805_2012Metric, F.Cu at (152.9, 88.0)
- added D4: LED, LED_SMD:LED_0805_2012Metric, F.Cu at (152.9, 90.0)
- added D5: LED, LED_SMD:LED_0805_2012Metric, F.Cu at (152.9, 92.0)
- added D6: LED, LED_SMD:LED_0805_2012Metric, F.Cu at (152.9, 94.0)
- added R6: 1K Ohms, Resistor_SMD:R_0805_2012Metric, F.Cu at (149.5, 88.0)
- added R7: 1K Ohms, Resistor_SMD:R_0805_2012Metric, F.Cu at (149.5, 90.0)
- added R8: 1K Ohms, Resistor_SMD:R_0805_2012Metric, F.Cu at (149.5, 92.0)
- added R9: 1K Ohms, Resistor_SMD:R_0805_2012Metric, F.Cu at (149.5, 94.0)
- added SW1: SW_Push, Button_Switch_THT:SW_PUSH_6mm_H5mm, F.Cu at (146.5, 69.5)
- moved U3 2.43 mm to (102.0, 86.5)
Connections:
- U1 pad 27: unconnected-(U1-PB1-Pad27) -> Net-(U1-PB1)
- U1 pad 28: unconnected-(U1-PB2-Pad28) -> Net-(U1-PB2)
- U1 pad 29: unconnected-(U1-PB10-Pad29) -> Net-(U1-PB10)
- U1 pad 30: unconnected-(U1-PB11-Pad30) -> Net-(U1-PB11)
Routing:
- net Buck-Boost Voltage: track 579.8 -> 642.5 mm, vias 27 -> 29
- net Net-(J5-Pin_1): track 1.70 -> 41.9 mm, vias 1 -> 5
- net Net-(J6-Pin_1): track 2.12 -> 25.1 mm, vias 1 -> 3
- net Net-(J8-Pin_1): track 1.95 -> 20.3 mm
- net Net-(J7-Pin_1): track 2.58 -> 20.3 mm
- net Net-(U1-PB1): track 0.00 -> 9.53 mm
- net Net-(U1-PB2): track 0.00 -> 8.15 mm
- net Net-(U1-PB10): track 0.00 -> 8.06 mm
- net unconnected-(U1-PB7-Pad59): track 0.00 -> 7.96 mm, vias 0 -> 1
- net unconnected-(U1-PB9-Pad62): track 0.00 -> 7.79 mm, vias 0 -> 1
- net Net-(U1-PB11): track 0.00 -> 7.76 mm
- net unconnected-(U1-PB6-Pad58): track 0.00 -> 7.75 mm, vias 0 -> 1
- net unconnected-(U1-PB8-Pad61): track 0.00 -> 7.38 mm, vias 0 -> 1
- net unconnected-(U2-RTCM-PadP$14): track 0.00 -> 7.03 mm, vias 0 -> 1
- net unconnected-(U2-NC@3-PadP$15): track 0.00 -> 7.03 mm, vias 0 -> 1
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Other:
- board text added: "BOOT"
- board text added: "Programming Pins"
- board text added: "RST"
- board text added: "SWCLK"
- board text added: "SWDIO"

Commit message: Schematic cleaned up
Parts:
- R4, R5: value 0 Ohms -> 0 Ohm
- moved R4 0.46 mm to (123.5, 89.5)
- moved R5 0.21 mm to (121.0, 82.0)
Connections:
- net Net-(C8-Pad1) renamed /Amp Out
- net Net-(D3-K) renamed +5V
- net Net-(J3-Pin_2) renamed /Speaker
- net Net-(J6-Pin_1) renamed /BOOT
- net Net-(J7-Pin_1) renamed /SWDIO
- net Net-(J8-Pin_1) renamed /SWCLK
- net Net-(U1-PA10) renamed /GPS TX
- net Net-(U1-PA4) renamed /DAC OUT
- net Net-(U1-PA9) renamed /GPS RX
- net Net-(U1-PB1) renamed /Debug 4
- net Net-(U1-PB10) renamed /Debug 2
- net Net-(U1-PB11) renamed /Debug 1
- net Net-(U1-PB2) renamed /Debug 3
- net Net-(U1-PC12) renamed /LoRa RX
- net Net-(U1-PD2) renamed /LoRa TX
- net Net-(U1-PH0) renamed /Clock
- net Net-(U8--) renamed /- Amp
- net Net-(U8-BYPASS) renamed /Bypass
- net VDDA Connection renamed /3.3VA
- C1 pad 1: Net-(D1-K) -> /Bat +
- C1 pad 2: Buck-Boost Voltage -> GND
- C10 pad 1: Buck-Boost Voltage -> +3.3V
- C10 pad 2: Buck-Boost Voltage -> GND
- C11 pad 2: Net-(U8-+) -> GND
- C12 pad 2: Buck-Boost Voltage -> GND
- C13 pad 1: Buck-Boost Voltage -> +3.3V
- C13 pad 2: Buck-Boost Voltage -> GND
- C14 pad 1: Buck-Boost Voltage -> +3.3V
- C14 pad 2: Buck-Boost Voltage -> GND
- C15 pad 1: Buck-Boost Voltage -> +3.3V
- C15 pad 2: Buck-Boost Voltage -> GND
- C16 pad 2: VDDA GND Connection -> /GNDA
- C17 pad 2: VDDA GND Connection -> /GNDA
- C18 pad 1: Buck-Boost Voltage -> +3.3V
- C18 pad 2: Buck-Boost Voltage -> GND
- C19 pad 1: Buck-Boost Voltage -> +3.3V
- C19 pad 2: Buck-Boost Voltage -> GND
- C2 pad 1: Buck-Boost Voltage -> +3.3V
- C2 pad 2: Buck-Boost Voltage -> GND
- C20 pad 1: Net-(J5-Pin_1) -> +3.3V
- C20 pad 2: Buck-Boost Voltage -> GND
- C3 pad 1: Net-(D1-K) -> /Bat +
- C3 pad 2: Buck-Boost Voltage -> GND
- C5 pad 2: Buck-Boost Voltage -> GND
- C6 pad 2: Buck-Boost Voltage -> GND
- C7 pad 2: Buck-Boost Voltage -> GND
- C8 pad 2: Buck-Boost Voltage -> GND
- D1 pad 1: Net-(D1-K) -> /Bat +
- D2 pad 1: Buck-Boost Voltage -> GND
- D3 pad 2: Net-(D1-K) -> Net-(D3-A)
- D4 pad 1: Buck-Boost Voltage -> GND
- D5 pad 1: Buck-Boost Voltage -> GND
- D6 pad 1: Buck-Boost Voltage -> GND
- J2 pad 1: Buck-Boost Voltage -> GND
- J3 pad 1: Buck-Boost Voltage -> GND
- L2 pad 1: Net-(D1-K) -> /Bat +
- L2 pad 2: Net-(D1-K) -> Net-(D3-A)
- R1 pad 1: Net-(D1-K) -> /Bat +
- R2 pad 2: Buck-Boost Voltage -> GND
- R4 pad 1: Buck-Boost Voltage -> +3.3V
- R5 pad 1: Buck-Boost Voltage -> GND
- R5 pad 2: VDDA GND Connection -> /GNDA
- SW1 pad 1: Buck-Boost Voltage -> GND
- SW1 pad 2: Net-(J5-Pin_1) -> +3.3V
- U1 pad 1: Buck-Boost Voltage -> +3.3V
- U1 pad 12: VDDA GND Connection -> GND
- U1 pad 18: Buck-Boost Voltage -> GND
- U1 pad 19: Buck-Boost Voltage -> +3.3V
- U1 pad 31: Buck-Boost Voltage -> GND
- U1 pad 32: Buck-Boost Voltage -> +3.3V
- U1 pad 47: Buck-Boost Voltage -> GND
- U1 pad 48: Buck-Boost Voltage -> +3.3V
- U1 pad 63: Buck-Boost Voltage -> GND
- U1 pad 64: Buck-Boost Voltage -> +3.3V
- U1 pad 7: Net-(J5-Pin_1) -> +3.3V
- U2 pad P$1: Buck-Boost Voltage -> +3.3V
- U2 pad P$12: Buck-Boost Voltage -> GND
- U2 pad P$19: Buck-Boost Voltage -> GND
- U2 pad P$3: Buck-Boost Voltage -> GND
- U2 pad P$4: Buck-Boost Voltage -> +3.3V
- U2 pad P$8: Buck-Boost Voltage -> GND
- U3 pad 1: Buck-Boost Voltage -> +3.3V
- U3 pad 2: Buck-Boost Voltage -> +3.3V
- U3 pad 6: Buck-Boost Voltage -> GND
- U4 pad 1: Buck-Boost Voltage -> +3.3V
- U4 pad 10: Buck-Boost Voltage -> +3.3V
- U4 pad 11: Buck-Boost Voltage -> GND
- U4 pad 3: Buck-Boost Voltage -> GND
- U4 pad 5: Net-(D1-K) -> /Bat +
- U4 pad 6: Net-(D1-K) -> /Bat +
- U4 pad 7: Net-(D1-K) -> /Bat +
- U4 pad 8: Net-(D1-K) -> /Bat +
- U4 pad 9: Buck-Boost Voltage -> GND
- U5 pad 1: Net-(D1-K) -> Net-(D3-A)
- U5 pad 2: Buck-Boost Voltage -> GND
- U5 pad 5: Net-(D1-K) -> /Bat +
- U8 pad 3: Net-(U8-+) -> GND
- U8 pad 4: Buck-Boost Voltage -> GND
- U9 pad 1: Buck-Boost Voltage -> +3.3V
- U9 pad 3: Buck-Boost Voltage -> GND
Routing:
- net Buck-Boost Voltage: track 642.5 -> 0.00 mm, vias 29 -> 0
- net GND: track 0.00 -> 467.5 mm, vias 0 -> 51
- net (no net): track 0.00 -> 120.8 mm
- net +3.3V: track 0.00 -> 94.7 mm, vias 0 -> 18
- net Net-(D1-K): track 69.9 -> 0.00 mm, vias 2 -> 0
- net /Bat +: track 0.00 -> 63.9 mm, vias 0 -> 2
- net Net-(J5-Pin_1): track 41.9 -> 0.00 mm, vias 5 -> 0
- net VDDA GND Connection: track 14.3 -> 0.00 mm, vias 35 -> 0
- net /GNDA: track 0.00 -> 9.80 mm
- net Net-(D3-A): track 0.00 -> 5.96 mm
- net Net-(U8-+): track 4.94 -> 0.00 mm
- added copper zone on B.Cu, net GND
- added copper zone on F.Cu, net GND
- removed copper zone on B.Cu, net VDDA GND Connection
- removed copper zone on F.Cu, net VDDA GND Connection

Commit message: pcb fix
Connections:
- net Net-(D1-A) renamed /Batteries
Routing:
- net +3.3V: track 94.7 -> 99.7 mm
Changed lines of the file:
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@@
 	(net 1 "Net-(U5-FB)")
 	(net 2 "unconnected-(U1-PA1-Pad15)")
-	(net 3 "Net-(D1-A)")
+	(net 3 "/Batteries")
 	(net 4 "Net-(U4-L1)")
 	(net 5 "Net-(U4-L2)")
@@
 			(layers "F.Cu" "F.Paste" "F.Mask")
 			(roundrect_rratio 0.25)
-			(net 3 "Net-(D1-A)")
+			(net 3 "/Batteries")
 			(pinfunction "Pin_2")
 			(pintype "passive")
@@
 			(size 1.0668 1.8542)
 			(layers "F.Cu" "F.Paste" "F.Mask")
-			(net 3 "Net-(D1-A)")
+			(net 3 "/Batteries")
 			(pinfunction "A")
 			(pintype "passive")
@@
 		(tags "resistor handsolder")
 		(property "Reference" "R5"
-			(at 0 1.65 360)
+			(at 0 1.65 0)
 			(layer "B.SilkS")
 			(effects
@@
 		)
 		(property "Value" "0 Ohm"
-			(at 0 -1.65 360)
+			(at 0 -1.65 0)
 			(layer "B.Fab")
 			(effects
@@
 		)
 		(fp_text user "${REFERENCE}"
-			(at 0 0 360)
+			(at 0 0 0)
 			(layer "B.Fab")
 			(effects
@@
 		(tags "resistor handsolder")
 		(property "Reference" "R4"
-			(at 0 1.65 360)
+			(at 0 1.65 0)
 			(layer "B.SilkS")
 			(effects
@@
 		)
 		(property "Value" "0 Ohm"
-			(at 0 -1.65 360)
+			(at 0 -1.65 0)
 			(layer "B.Fab")
 			(effects
@@
 		)
 		(fp_text user "${REFERENCE}"
-			(at 0 0 360)
+			(at 0 0 0)
 			(layer "B.Fab")
 			(effects
@@
 	)
 	(segment
-		(start 117.61124 89.705902)
-		(end 117.613019 89.704123)
+		(start 122.5 89.5)
+		(end 117.817142 89.5)
 		(width 0.25)
 		(layer "B.Cu")
@@
 		(width 0.25)
 		(layer "B.Cu")
+		(net 70)
+	)
+	(segment
+		(start 117.817142 89.5)
+		(end 117.61124 89.705902)
+		(width 0.25)
+		(layer "B.Cu")

Commit message: minor pcb changes
Parts:
- added R10: 100k Ohms, Resistor_SMD:R_0805_2012Metric, F.Cu at (133.7, 60.5)
- added R11: 100k Ohms, Resistor_SMD:R_0805_2012Metric, F.Cu at (133.7, 63.5)
- C9: value 1000 uF -> 100 uF
Connections:
- C20 pad 1: +3.3V -> /RST
- SW1 pad 2: +3.3V -> /RST
- U1 pad 12: GND -> /GNDA
- U1 pad 7: +3.3V -> /RST
Routing:
- net +3.3V: track 99.7 -> 57.8 mm, vias 18 -> 13
- net /RST: track 0.00 -> 41.9 mm, vias 0 -> 5
- net GND: track 467.5 -> 463.3 mm, vias 51 -> 50
- net /GNDA: track 9.80 -> 14.0 mm, vias 0 -> 1

Commit message: minor pcb tweaks
Parts:
- removed REF** (x4): MountingHole_2.2mm_M2, MountingHole:MountingHole_2.2mm_M2
- added J5: Conn_01x04_Pin, Connector_JST:JST_EH_B4B-EH-A_1x04_P2.50mm_Vertical, F.Cu at (178.9, 85.0)
- C11, C12, C20, D1, R10, R11: moved to B.Cu
- C18: moved to F.Cu
- C9: footprint Polarized Cap 1000 uF:PCAP_10x10-ELECT_NCA -> Polarized Caps (.1 - 100 uF):CAP_UZE_4X3P9_NCH
- R1, R2, R3: footprint Resistor_SMD:R_0805_2012Metric -> Resistor_SMD:R_0805_2012Metric_Pad1.20x1.40mm_HandSolder
- U4: footprint Buck-Boost:DRC0010J -> Buck-Boost Converter Chip:DRC0010J
- U5: footprint Boost:MF05A -> Boost Converter Chip:MF05A
- moved J2 86.8 mm to (131.5, 28.5), turned to 180 degrees
- moved C4 80.4 mm to (115.5, 36.5), turned to 180 degrees
- moved R2 76.8 mm to (120.0, 36.5), turned to 0 degrees
- moved L2 76.6 mm to (113.3, 31.0)
- moved R3 76.2 mm to (115.6, 39.5), turned to 180 degrees
- moved U5 71.3 mm to (120.0, 41.0), turned to -90 degrees
- moved C5 70.7 mm to (125.0, 45.0)
- moved D1 69.4 mm to (129.0, 37.6), turned to 90 degrees
- moved D3 68.0 mm to (125.5, 35.9), turned to 90 degrees
- moved R1 67.8 mm to (115.5, 44.0)
- moved C1 67.7 mm to (138.5, 37.2), turned to 180 degrees
- moved J3 66.9 mm to (126.5, 83.0), turned to 0 degrees
- moved C3 63.3 mm to (110.5, 46.0), turned to 180 degrees
- moved C12 63.0 mm to (114.0, 73.0), turned to 180 degrees
- moved C9 63.0 mm to (123.5, 75.5)
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Connections:
- net Net-(D2-A) renamed /D1LED
- net Net-(D3-A) renamed /SW Boost
- net Net-(D4-A) renamed /D2LED
- net Net-(D5-A) renamed /D3LED
- net Net-(D6-A) renamed /D4LED
- net Net-(U4-L1) renamed /L1 Buck
- net Net-(U4-L2) renamed /L2 Buck
- net Net-(U5-EN) renamed /EN Boost
- net Net-(U5-FB) renamed /FB Boost
Routing:
- net GND: track 463.3 -> 105.9 mm, vias 50 -> 21
- net (no net): track 120.8 -> 0.00 mm
- net /LoRa TX: track 53.1 -> 0.00 mm, vias 2 -> 0
- net /LoRa RX: track 47.7 -> 0.00 mm, vias 1 -> 0
- net /Bat +: track 63.9 -> 33.3 mm, vias 2 -> 4
- net /DAC OUT: track 27.8 -> 0.00 mm
- net /GPS RX: track 24.2 -> 0.00 mm, vias 1 -> 0
- net /GPS TX: track 23.8 -> 0.00 mm, vias 1 -> 0
- net +5V: track 51.2 -> 28.2 mm, vias 2 -> 3
- net /RST: track 41.9 -> 19.1 mm, vias 5 -> 0
- net /BOOT: track 25.1 -> 3.41 mm, vias 3 -> 1
- net /SWDIO: track 20.3 -> 0.00 mm, vias 1 -> 0
- net /SWCLK: track 20.3 -> 0.00 mm, vias 1 -> 0
- net /FB Boost: track 21.0 -> 8.73 mm, vias 0 -> 1
- net /Debug 4: track 9.53 -> 0.00 mm
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- added copper zone on F.Cu, net +3.3V
- added copper zone on F.Cu, net +5V
- added copper zone on F.Cu, net /Bat +
- added copper zone on F.Cu, net /L1 Buck
- added copper zone on F.Cu, net /L2 Buck
- added copper zone on F.Cu, net /SW Boost
Other:
- board outline removed
- board text removed: "BOOT"
- board text removed: "Connectors"
- board text removed: "ECE 477 Team 5: Smart Dog Collar Andrew Wu David Manojlovic Nick Durnil Ethan James Revision: Version 1"
- board text removed: "GPS Signal Connections (TX & RX)"
- board text removed: "LM2735 Boost Chip"
- board text removed: "LM386 Amplifier Chip"
- board text removed: "LoRa Signal Connections (TX & RX)"
- board text removed: "MTK MT3339 GPS Chip"
- board text removed: "Pin 1"
- board text removed: "Programming Pins"
- board text removed: "RST"
- board text removed: "RYLR896 LoRa Chip"
- board text removed: "STM32L4"
- board text removed: "SWCLK"
- board text removed: "SWDIO"
- board text removed: "TPS63 Buck-Boost Chip"
