File: PCB/PCB.kicad_pcb (KiCad board)
At the start: 2 copper layers, 64.8 x 61 mm, 54 parts, among them J2 Conn_01x02_Pin, J3 Conn_01x02_Pin, J5 Conn_01x04_Pin, SW1 SW_Push, U1 STM32L476RGTx, U2 FGPMMOPA6H, U4 TPS63001DRCR, U5 LM2735XMF/NOPB, U8 LM386, U9 MAX7375AXR805

Commit message: gbr file fixes
Routing:
- net /Bypass: track 8.21 -> 8.98 mm
- net GND: track 125.5 -> 125.7 mm, vias 59 -> 61
Changed lines of the file:
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@@
 			(drillshape 0)
 			(scaleselection 1)
-			(outputdirectory "")
+			(outputdirectory "gbr files/")
 		)
 	)
@@
 	)
 	(gr_text "ECE 477 Team 5: Smart Dog Collar\nAndrew Wu\nNick Durnil\nDavid Manojlovic\nEthan James\nVersion 5"
-		(at 215.9 140.97 0)
+		(at 214.56 143.09 0)
 		(layer "F.SilkS")
 		(effects
 			(font
-				(size 0.5 0.5)
+				(size 0.75 0.75)
 				(thickness 0.1)
 				(bold yes)
@@
 	)
 	(segment
-		(start 187.5 100.2418)
-		(end 188 100.2418)
-		(width 0.254)
+		(start 225.815 116.595)
+		(end 225.815 120.23)
+		(width 0.25)
 		(layer "F.Cu")
 		(net 2)
 	)
 	(segment
-		(start 225.815 116.595)
-		(end 225.815 120.23)
-		(width 0.25)
+		(start 184 100.2418)
+		(end 183.38685 100.2418)
+		(width 0.5)
 		(layer "F.Cu")
 		(net 2)
@@
 	)
 	(segment
+		(start 183.38685 100.2418)
+		(end 183.385377 100.240327)
+		(width 0.5)
+		(layer "F.Cu")
+		(net 2)
+	)
+	(segment
 		(start 173.7253 114.2747)
 		(end 174 114)
@@
 	)
 	(via
+		(at 182.49 100.61)
+		(size 0.8)
+		(drill 0.4)
+		(layers "F.Cu" "B.Cu")
+		(free yes)
+		(net 2)
+	)
+	(via
 		(at 229.87 101.6)
 		(size 0.8)
@@
 	)
 	(via
+		(at 188.01 100.84)
+		(size 0.8)
+		(drill 0.4)
+		(layers "F.Cu" "B.Cu")
+		(free yes)
+		(net 2)
+	)
+	(via
 		(at 215.9 93.98)
 		(size 0.8)
@@
 	)
 	(segment
+		(start 178.1663 122.2863)
+		(end 178.1663 123.6)
+		(width 0.25)
+		(layer "F.Cu")
+		(net 21)
+	)
+	(segment
 		(start 180.42 124.54)
 		(end 181.325305 124.54)
@@
 	)
 	(segment
+		(start 179.48 123.6)
+		(end 180.42 124.54)
+		(width 0.25)
+		(layer "F.Cu")
+		(net 21)
+	)
+	(segment
 		(start 183.435 126.649695)
 		(end 183.435 127.26415)
@@
 	(segment
 		(start 177.8 121.92)
-		(end 180.42 124.54)
+		(end 178.1663 122.2863)
+		(width 0.25)
+		(layer "F.Cu")
+		(net 21)
+	)
+	(segment
+		(start 178.1663 123.6)
+		(end 179.48 123.6)
 		(width 0.25)
 		(layer "F.Cu")
