File: PCB/PCB.kicad_sch (KiCad schematic)
At the start: 60 parts, among them J1 Conn_01x02_Socket, J2 Conn_01x02_Pin, J3 Conn_01x02_Pin, J4 Conn_01x02_Socket, J5 Conn_01x04_Pin, SW1 SW_Push, U1 STM32L476RGTx, U2 FGPMMOPA6H, U4 TPS63001DRCR, U5 LM2735XMF/NOPB, U8 LM386, U9 MAX7375AXR805

Commit message: pcb v5
Connections:
- net GND: no longer C11.2, U8.3 (+)
- new net Amp In: C11.2, U8.3 (+)
Other:
- moved on the sheet: C11
Changed lines of the file:
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@@
 	)
 	(junction
-		(at 218.44 102.87)
-		(diameter 0)
-		(color 0 0 0 0)
-	)
-	(junction
 		(at 243.84 41.91)
 		(diameter 0)
@@
 	(wire
 		(pts
-			(xy 218.44 96.52) (xy 218.44 102.87)
+			(xy 218.44 96.52) (xy 218.44 107.95)
 		)
 		(stroke
@@
 	(wire
 		(pts
-			(xy 218.44 102.87) (xy 229.87 102.87)
+			(xy 217.17 102.87) (xy 229.87 102.87)
 		)
 		(stroke
@@
 	(wire
 		(pts
-			(xy 203.2 102.87) (xy 210.82 102.87)
+			(xy 203.2 102.87) (xy 209.55 102.87)
 		)
 		(stroke
@@
 	(wire
 		(pts
-			(xy 218.44 102.87) (xy 218.44 107.95)
-		)
-		(stroke
-			(width 0)
-			(type default)
-		)
-	)
-	(wire
-		(pts
 			(xy 3.81 -8.89) (xy -2.54 -8.89)
 		)
@@
 	(symbol
 		(lib_id "Device:C")
-		(at 214.63 102.87 90)
+		(at 213.36 102.87 90)
 		(unit 1)
 		(exclude_from_sim no)
@@
 		(fields_autoplaced yes)
 		(property "Reference" "C11"
-			(at 214.63 96.52 90)
+			(at 213.36 96.52 90)
 			(effects
 				(font
@@
 		)
 		(property "Value" ".1 uF"
-			(at 214.63 99.06 90)
+			(at 213.36 99.06 90)
 			(effects
 				(font
@@
 		)
 		(property "Footprint" "Capacitor_SMD:C_0805_2012Metric_Pad1.18x1.45mm_HandSolder"
-			(at 218.44 101.9048 0)
+			(at 217.17 101.9048 0)
 			(effects
 				(font
@@
 		)
 		(property "Datasheet" "~"
-			(at 214.63 102.87 0)
+			(at 213.36 102.87 0)
 			(effects
 				(font
@@
 		)
 		(property "Description" ""
-			(at 214.63 102.87 0)
+			(at 213.36 102.87 0)
 			(effects
 				(font
